Commit message: some change for test, add ros::spin() in waypoint_publisher.cpp otherwise it won't takeoff,add some arg in spawn_mav_tbm_2.launch make it can create  gazebo plugin with I wanted namespace

File: rotors_description/urdf/component_snippets.xacro (robot description, xacro)
@@ -249,5 +249,6 @@
   <!-- ==================== ROS INTERFACE MACRO ====================== -->
   <!-- =============================================================== -->
-  <!-- <xacro:macro
+  <!--
+  <xacro:macro
   		name="ros_interface_plugin_macro"
   		params="namespace">
@@ -257,5 +258,6 @@
       </plugin>
     </gazebo>
-  </xacro:macro>-->
+  </xacro:macro>
+	-->
   <!-- =============================================================== -->
   <!-- ================== MAVLINK INTERFACE MACRO ==================== -->

File: rotors_description/urdf/firefly_base.xacro (robot description, xacro)
@@ -23,5 +23,5 @@
   <xacro:controller_plugin_macro namespace="${namespace}" imu_sub_topic="imu" />
   <!-- Instantiate a ROS message interface -->
-  <!-- <xacro:ros_interface_plugin_macro namespace="${namespace}" />-->
+   <!-- <xacro:ros_interface_plugin_macro namespace="${namespace}" /> -->
   <xacro:if value="$(arg enable_mavlink_interface)">
     <!-- Instantiate mavlink telemetry interface. -->
